File: project_02/EAGLE/ENGI301_Project-2.sch (EAGLE design)
At the start: 18 parts, among them U1 POCKETBEAGLE, U2 MIKROE_CLICKLARGE

Commit message: Updates
Other:
- note added: "1"
- note added: "Theodore Hoisington"
Changed lines of the file:
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@@
 <wire x1="10.16" y1="63.5" x2="119.38" y2="63.5" width="0.8128" layer="97"/>
 <text x="15.24" y="53.34" size="5.08" layer="97">Mounting Holes and Fiducials</text>
+<text x="313.436" y="20.32" size="2.286" layer="94">Theodore Hoisington</text>
+<text x="325.12" y="5.08" size="2.286" layer="94">1</text>
 </plain>
 <instances>
